Commit message: Add files via upload

File: src/mybot_description/urdf/mybot.xacro (robot description, xacro)
@@ -25,5 +25,5 @@
       <origin xyz="0 0 0.1" rpy=" 0 0 0"/>
       <geometry>
-        <mesh filename="$(find mybot_description)/meshes/chassis.dae"/>
+        <mesh filename="package://mybot_description/meshes/chassis.dae"/>
       </geometry>
     </visual>
@@ -49,4 +49,5 @@
         <sphere radius="0.05"/>
       </geometry>
+	<material name="black"/>
     </visual>
   </link>
@@ -64,4 +65,5 @@
         <cylinder radius="0.1" length="0.05"/>
       </geometry>
+	<material name="black"/>
     </visual>
     <inertial>
@@ -88,4 +90,5 @@
         <cylinder radius="0.1" length="0.05"/>
       </geometry>
+	<material name="black"/>
     </visual>
     <inertial>
